Commit message: Update ros2  Ackermann packages

File: recipes-ros2packages/ackermann-description/files/ackermann_description/urdf/base.xacro (robot description, xacro)
@@ -25,5 +25,5 @@
   <xacro:property name="wheel_inertia_izz" value="${1.0/12.0 * wheel_mass * (3*wheel_radius*wheel_radius + wheel_width*wheel_width)}"/>
   <xacro:property name="steering_velocity_max" value="1.0"/>
-  <xacro:property name="steering_max" value="0.373302"/> <!-- 21.38 degrees-->
+  <xacro:property name="steering_max" value="0.2421"/>
   <xacro:property name="wheel_effort_max" value="0.206"/> <!-- load torque in nm -->
   <xacro:property name="wheel_velocity_max" value="15.38"/> <!-- 0.5 m/s with r=0.0325m -->

File: recipes-ros2packages/ackermann-description/files/ackermann_description/urdf/sensors.xacro (robot description, xacro)
@@ -26,5 +26,5 @@
         <parent link="base_link"/>
         <child link="camera_link"/>
-        <origin xyz="0.23 0 0.1" rpy="0 0 0"/>
+        <origin xyz="0.25 0 0.099" rpy="0 0 0"/>
     </joint>
     <!-- ====== CAMERA OPTICAL LINK ====== -->
@@ -96,5 +96,5 @@
         <parent link="base_link"/>
         <child link="lidar_link"/>
-        <origin xyz="0.125 0 0.195" rpy="0 0 ${pi}"/>
+        <origin xyz="0.22 0 0.279" rpy="0 0 0"/>
     </joint>
     <!-- ====== LIDAR GAZEBO ======= -->
@@ -140,6 +140,5 @@
      <xacro:include filename="$(find ros2_livox_simulation)/urdf/mid360.xacro" />
     <xacro:mid360 name="livox" parent="base_link" topic="mid360">
-        <!-- Same mounting position as your old lidar; remove ${pi} yaw if the mesh is already oriented forward -->
-        <origin xyz="0.125 0 0.195" rpy="0 0 0"/>
+        <origin xyz="0.22 0 0.279" rpy="0 0 0"/>
     </xacro:mid360>
     </xacro:unless>
@@ -169,5 +168,5 @@
         <parent link="base_link"/>
         <child link="imu_link"/>
-        <origin xyz="0.117 0.06 0.05" rpy="0 0 0"/>
+        <origin xyz="0.092 -0.03 0.018" rpy="0 0 0"/>
     </joint>
     <!-- ====== IMU GAZEBO  ====== -->
