Commit message: Fix dead TF publish

File: recipes-ros2packages/ackermann-description/files/ackermann_description/urdf/sensors.xacro (robot description, xacro)
@@ -96,5 +96,5 @@
         <parent link="base_link"/>
         <child link="lidar_link"/>
-        <origin xyz="0.22 0 0.279" rpy="0 0 0"/>
+        <origin xyz="0.15 0 0.279" rpy="0 0 0"/>
     </joint>
     <!-- ====== LIDAR GAZEBO ======= -->

Commit message: Add Some Ackermann fixes & recipes for testing

File: recipes-ros2packages/ackermann-description/files/ackermann_description/urdf/sensors.xacro (robot description, xacro)
@@ -98,4 +98,13 @@
         <origin xyz="0.15 0 0.279" rpy="0 0 0"/>
     </joint>
+    <!-- Frame for the Mid-360 internal IMU, which publishes /livox/imu.
+         PROVISIONAL OFFSET - identity is a placeholder, not the real extrinsic.
+         Replace with the measured value before trusting any LIO result. -->
+    <link name="livox_frame"/>
+    <joint name="livox_imu_joint" type="fixed">
+        <parent link="lidar_link"/>
+        <child link="livox_frame"/>
+        <origin xyz="0 0 0" rpy="0 0 0"/>
+    </joint>
     <!-- ====== LIDAR GAZEBO ======= -->
      <gazebo reference="lidar_link">

Commit message: Modify Lidar Link

File: recipes-ros2packages/ackermann-description/files/ackermann_description/urdf/sensors.xacro (robot description, xacro)
@@ -96,5 +96,5 @@
         <parent link="base_link"/>
         <child link="lidar_link"/>
-        <origin xyz="0.15 0 0.279" rpy="0 0 0"/>
+        <origin xyz="0.13 0 0.279" rpy="0 0 0"/>
     </joint>
     <!-- Frame for the Mid-360 internal IMU, which publishes /livox/imu.
